File: pcb/michibot.brd (EAGLE design)
At the start: 68 x 93.4 mm, 20 parts, among them U1 RASPBERRY_PICOSMD-TH, U2 GY-521MPU6050

Commit message: idk, but just in case:)
Connections:
- removed net 3V3(OUT): U1.36, U1.P$36
- removed net 3V3@1: U$1.1, U$1.3, U1.39, U1.P$39
- removed net GND: U1.13, U1.18, U1.23, U1.28, U1.3, U1.33, U1.38, U1.8, U1.P$13, U1.P$18, U1.P$23, U1.P$28, U1.P$3, U1.P$33, U1.P$38, U1.P$8
- new net 5V0@1: U$1.2, U$2.OUT+, U1.39, U1.P$39
- new net GND@8: U$1.6, U$2.OUT-, U1.13, U1.18, U1.23, U1.28, U1.3, U1.33, U1.38, U1.8, U1.P$13, U1.P$18, U1.P$23, U1.P$28, U1.P$3, U1.P$33, U1.P$38, U1.P$8, U2.GND
- new net N$1: U1.36, U1.P$36, U2.VCC
- new net N$10: U$9.3, U1.6, U1.P$6
- new net N$11: U$5.3, U1.7, U1.P$7
- new net N$12: U$14.3, U1.9, U1.P$9
- new net N$13: U$10.3, U1.10, U1.P$10
- new net N$14: U$6.3, U1.11, U1.P$11
- new net N$15: U$11.3, U1.12, U1.P$12
- new net N$16: U$7.3, U1.14, U1.P$14
- new net N$4: CN1.1, U$2.IN+, U$3.IN+
- new net N$5: CN1.2, U$2.IN-, U$3.IN-
- new net N$6: U$13.3, U1.5, U1.P$5
- new net N$7: U$12.3, U1.1, U1.P$1
- new net N$8: U$8.3, U1.2, U1.P$2
- new net N$9: U$4.3, U1.4, U1.P$4
Routing:
- net 3V3@1: track 17.5 -> 0.00 mm
