File: pcb/michibot.sch (EAGLE design)
At the start: 20 parts, among them U1 RASPBERRY_PICOSMD-TH, U2 GY-521MPU6050

Commit message: idk, but just in case:)
Connections:
- removed net 3V3@1: U$1.3V3@1, U$1.GPIO2/SDA1, U1.VSYS
- new net 5V0@1: U$1.5V0@1, U$2.OUT+, U1.VSYS
- new net GND@8: U$1.GND@8, U$2.OUT-, U1.GND, U2.GND
- new net N$1: U1.3V3(OUT), U2.VCC
- new net N$10: U$9.S, U1.GP4
- new net N$11: U$5.S, U1.GP5
- new net N$12: U$14.S, U1.GP6
- new net N$13: U$10.S, U1.GP7
- new net N$14: U$6.S, U1.GP8
- new net N$15: U$11.S, U1.GP9
- new net N$16: U$7.S, U1.GP10
- new net N$4: CN1.2, U$2.IN+, U$3.IN+
- new net N$5: CN1.1, U$2.IN-, U$3.IN-
- new net N$6: U$13.S, U1.GP3
- new net N$7: U$12.S, U1.GP0
- new net N$8: U$8.S, U1.GP1
- new net N$9: U$4.S, U1.GP2
Other:
- moved on the sheet: CN1, LED3, U$10, U$11, U$12, U$13, U$14, U$4, U$5, U$6, U$7, U$8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
